File: DCDC_5V.kicad_sch (KiCad schematic)
At the start: 12 parts, among them U10 TPS563200

Commit message: Add option 12V Elec + add missing brake pullups
Changed lines of the file:
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@@
 (kicad_sch
-	(version 20231120)
+	(version 20250114)
 	(generator "eeschema")
-	(generator_version "8.0")
+	(generator_version "9.0")
 	(paper "A4")
 	(junction

Commit message: various updates
Parts:
- C21, C22: LCSC# C1713 -> C440198
Changed lines of the file:
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@@
 			)
 		)
-		(property "LCSC#" "C1713"
+		(property "LCSC#" "C440198"
 			(at 87.63 78.74 0)
 			(effects
@@
 			)
 		)
-		(property "LCSC#" "C1713"
+		(property "LCSC#" "C440198"
 			(at 97.79 78.74 0)
 			(effects

Commit message: change capacitor references to support >25V
Parts:
- C24, C25: LCSC# C5674 -> C29277
Changed lines of the file:
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@@
 			)
 		)
-		(property "LCSC#" "C5674"
+		(property "LCSC#" "C29277"
 			(at 187.96 80.01 0)
 			(effects
@@
 			)
 		)
-		(property "LCSC#" "C5674"
+		(property "LCSC#" "C29277"
 			(at 198.12 80.01 0)
 			(effects
